File: frontend-prot.kicad_sch (KiCad schematic)
At the start: 37 parts, among them J5 IN, J6 LO, Q1 MMBT6520L, Q2 MMBT6520L, Q3 MMBT6520L, Q4 MMBT6520L, Q5 MMBT6520L, Q6 MMBT6520L, Q7 MMBT6520L, Q8 MMBT6520L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

Commit message: small changes, add missing part numbers
Parts:
- SW4: value SW_DPDT_x2 -> G6KU-2F-Y; footprint (none) -> Relay_SMD:Relay_DPDT_Omron_G6K-2F-Y
Connections:
- net GND: now also SW4.4 (A); no longer SW4.6 (C)
- net at L1.2, SW4.1 (A): now also SW4.6 (C); no longer SW4.4 (A)
Other:
- moved on the sheet: SW4B
Changed lines of the file:
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@@
 	(symbol
 		(lib_id "Switch:SW_DPDT_x2")
-		(at 149.86 85.09 0)
-		(mirror y)
+		(at 149.86 85.09 180)
 		(unit 2)
 		(exclude_from_sim no)
@@
 		(on_board yes)
 		(dnp no)
-		(fields_autoplaced yes)
 		(property "Reference" "SW4"
 			(at 149.86 76.2 0)
@@
 			)
 		)
-		(property "Value" "SW_DPDT_x2"
+		(property "Value" "G6KU-2F-Y"
 			(at 149.86 78.74 0)
 			(effects
@@
 			)
 		)
-		(property "Footprint" ""
+		(property "Footprint" "Relay_SMD:Relay_DPDT_Omron_G6K-2F-Y"
 			(at 149.86 85.09 0)
 			(effects
@@
 			)
 		)
-		(property "Datasheet" "~"
+		(property "Datasheet" "https://omronfs.omron.com/en_US/ecb/products/pdf/en-g6k.pdf"
 			(at 149.86 85.09 0)
 			(effects
@@
 			)
 		)
-		(property "Value" "SW_DPDT_x2"
+		(property "Value" "G6KU-2F-Y"
 			(at 149.86 60.96 0)
 			(effects
@@
 			)
 		)
-		(property "Footprint" ""
+		(property "Footprint" "Relay_SMD:Relay_DPDT_Omron_G6K-2F-Y"
 			(at 149.86 67.31 0)
 			(effects
@@
 			)
 		)
-		(property "Datasheet" "~"
+		(property "Datasheet" "https://omronfs.omron.com/en_US/ecb/products/pdf/en-g6k.pdf"
 			(at 149.86 67.31 0)
 			(effects
